File: breadbee.kicad_pcb (KiCad board)
At the start: 4 copper layers, 32 x 30 mm, 83 parts, among them J1 HR961160C, J2 Conn_02x12_Odd_Even, J3 USB_B_Micro, J4 Conn_01x21, U1 msc313e, U2 spinor, U3 ea3036c, U4 ch340e, U5 tvsarray, Y1 Crystal_GND24

Commit message: Fix screw up with the sar pins
Parts:
- C1, C11, C12, C13, C14, C15, C18, C19, C20, C21, C22, C24, C25, C26, C35, C36, C37, C38, C6: value C -> 1uf
- C2, C3, C4: value C -> 220pf
- C28, C30, C31, C32: value C -> 10uf
- C33, C34: value C -> 100nf
- C7, C8: value C -> 18pf
- R1: value R -> 200k
- R13, R14, R15, R16: value R -> 22
- R18, R2, R21, R22, R3: value R -> 100k
- R19, R20, R8: value R -> 1m
- R23: value R -> 1.2m
- R4: value R -> 150k
- R5: value R -> 510k
- R6: value R -> 110K
- R7: value R -> 1.1m
Connections:
- J2 pad 11: /sar_gpio1 -> /sar_gpio2
- J2 pad 12: /sar_gpio0 -> /sar_gpio3
- J2 pad 13: /sar_gpio2 -> /sar_gpio1
- J2 pad 14: /sar_gpio3 -> /sar_gpio0
- U1 pad 10: /sar_gpio1 -> /sar_gpio2
- U1 pad 11: /sar_gpio2 -> /sar_gpio1
- U1 pad 12: /sar_gpio3 -> /sar_gpio0
- U1 pad 9: /sar_gpio0 -> /sar_gpio3
Routing:
- net /sar_gpio3: track 6.62 -> 5.71 mm
- net /sar_gpio0: track 5.71 -> 6.62 mm

Commit message: Fix solder mask.
Other:
- rule pad_to_mask_clearance: 0.051 -> 0
- rule solder_mask_min_width: 0.25 -> 0.01
Changed lines of the file:
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@@
-(kicad_pcb (version 20171130) (host pcbnew 5.1.2+dfsg1-1)
+(kicad_pcb (version 20171130) (host pcbnew 5.1.4+dfsg1-1)
   (general
     (thickness 1.6)
@@
     (pad_size 1.524 1.524)
     (pad_drill 0.762)
-    (pad_to_mask_clearance 0.051)
-    (solder_mask_min_width 0.25)
+    (pad_to_mask_clearance 0)
+    (solder_mask_min_width 0.01)
     (aux_axis_origin 0 0)
     (grid_origin 141.48 83.93)
@@
   (segment (start 133.098 98.916) (end 134.808932 98.916) (width 0.1545) (layer B.Cu) (net 28))
   (segment (start 134.808932 98.916) (end 135.253432 99.3605) (width 0.1545) (layer B.Cu) (net 28))
-  (segment (start 143.1917 98.9683) (end 142.549999 99.610001) (width 0.1545) (layer F.Cu) (net 32) (status 20))
-  (segment (start 143.1917 97.329338) (end 143.1917 98.9683) (width 0.1545) (layer F.Cu) (net 32))
-  (segment (start 142.549999 99.610001) (end 141.7 100.46) (width 0.1545) (layer F.Cu) (net 32) (status 30))
-  (segment (start 142.770451 96.908089) (end 143.1917 97.329338) (width 0.1545) (layer F.Cu) (net 32))
-  (segment (start 142.770451 96.723383) (end 142.770451 96.908089) (width 0.1545) (layer F.Cu) (net 32))
-  (segment (start 142.665 96.617932) (end 142.770451 96.723383) (width 0.1545) (layer F.Cu) (net 32))
-  (segment (start 142.665 95.59) (end 142.665 96.617932) (width 0.1545) (layer F.Cu) (net 32) (status 10))
+  (segment (start 143.715 96.658296) (end 143.715 95.59) (width 0.1545) (layer F.Cu) (net 29) (status 20))
+  (segment (start 144.042529 96.985827) (end 143.715 96.658296) (width 0.1545) (layer F.Cu) (net 29))
+  (segment (start 144.24 100.46) (end 144.24 99.257919) (width 0.1545) (layer F.Cu) (net 29) (status 10))
+  (segment (start 144.042529 99.060448) (end 144.042529 96.985827) (width 0.1545) (layer F.Cu) (net 29))
+  (segment (start 144.24 99.257919) (end 144.042529 99.060448) (width 0.1545) (layer F.Cu) (net 29))
+  (segment (start 143.715 96.658299) (end 144.042527 96.985826) (width 0.1545) (layer F.Cu) (net 29))
+  (segment (start 143.715 95.59) (end 143.715 96.658299) (width 0.1545) (layer F.Cu) (net 29) (status 10))
+  (segment (start 143.365 96.1195) (end 143.365 95.59) (width 0.1545) (layer F.Cu) (net 30) (status 20))
+  (segment (start 144.24 103) (end 143.15151 101.91151) (width 0.1545) (layer F.Cu) (net 30) (status 10))
+  (segment (start 143.15151 101.91151) (end 143.15151 99.818488) (width 0.1545) (layer F.Cu) (net 30))
+  (segment (start 143.15151 99.818488) (end 143.761018 99.20898) (width 0.1545) (layer F.Cu) (net 30))
+  (segment (start 143.43349 96.18799) (end 143.365 96.1195) (width 0.1545) (layer F.Cu) (net 30))
+  (segment (start 143.761018 97.102431) (end 143.43349 96.774903) (width 0.1545) (layer F.Cu) (net 30))
+  (segment (start 143.43349 96.774903) (end 143.43349 96.18799) (width 0.1545) (layer F.Cu) (net 30))
+  (segment (start 143.761018 99.20898) (end 143.761018 97.102431) (width 0.1545) (layer F.Cu) (net 30))
   (segment (start 142.869999 101.830001) (end 142.549999 102.150001) (width 0.1545) (layer F.Cu) (net 31) (status 20))
   (segment (start 142.869999 99.701883) (end 142.869999 101.830001) (width 0.1545) (layer F.Cu) (net 31))
@@
   (segment (start 143.151979 96.891509) (end 143.479507 97.219036) (width 0.1545) (layer F.Cu) (net 31))
   (segment (start 143.479507 99.092375) (end 142.869999 99.701883) (width 0.1545) (layer F.Cu) (net 31))
-  (segment (start 143.365 96.1195) (end 143.365 95.59) (width 0.1545) (layer F.Cu) (net 30) (status 20))
-  (segment (start 144.24 103) (end 143.15151 101.91151) (width 0.1545) (layer F.Cu) (net 30) (status 10))
-  (segment (start 143.15151 101.91151) (end 143.15151 99.818488) (width 0.1545) (layer F.Cu) (net 30))
-  (segment (start 143.15151 99.818488) (end 143.761018 99.20898) (width 0.1545) (layer F.Cu) (net 30))
-  (segment (start 143.43349 96.18799) (end 143.365 96.1195) (width 0.1545) (layer F.Cu) (net 30))
-  (segment (start 143.761018 97.102431) (end 143.43349 96.774903) (width 0.1545) (layer F.Cu) (net 30))
-  (segment (start 143.43349 96.774903) (end 143.43349 96.18799) (width 0.1545) (layer F.Cu) (net 30))
-  (segment (start 143.761018 99.20898) (end 143.761018 97.102431) (width 0.1545) (layer F.Cu) (net 30))
-  (segment (start 143.715 96.658296) (end 143.715 95.59) (width 0.1545) (layer F.Cu) (net 29) (status 20))
-  (segment (start 144.042529 96.985827) (end 143.715 96.658296) (width 0.1545) (layer F.Cu) (net 29))
-  (segment (start 144.24 100.46) (end 144.24 99.257919) (width 0.1545) (layer F.Cu) (net 29) (status 10))
-  (segment (start 144.042529 99.060448) (end 144.042529 96.985827) (width 0.1545) (layer F.Cu) (net 29))
-  (segment (start 144.24 99.257919) (end 144.042529 99.060448) (width 0.1545) (layer F.Cu) (net 29))
-  (segment (start 143.715 96.658299) (end 144.042527 96.985826) (width 0.1545) (layer F.Cu) (net 29))
-  (segment (start 143.715 95.59) (end 143.715 96.658299) (width 0.1545) (layer F.Cu) (net 29) (status 10))
+  (segment (start 143.1917 98.9683) (end 142.549999 99.610001) (width 0.1545) (layer F.Cu) (net 32) (status 20))
+  (segment (start 143.1917 97.329338) (end 143.1917 98.9683) (width 0.1545) (layer F.Cu) (net 32))
+  (segment (start 142.549999 99.610001) (end 141.7 100.46) (width 0.1545) (layer F.Cu) (net 32) (status 30))
+  (segment (start 142.770451 96.908089) (end 143.1917 97.329338) (width 0.1545) (layer F.Cu) (net 32))
+  (segment (start 142.770451 96.723383) (end 142.770451 96.908089) (width 0.1545) (layer F.Cu) (net 32))
+  (segment (start 142.665 96.617932) (end 142.770451 96.723383) (width 0.1545) (layer F.Cu) (net 32))
+  (segment (start 142.665 95.59) (end 142.665 96.617932) (width 0.1545) (layer F.Cu) (net 32) (status 10))
   (via (at 149.151206 88.751332) (size 0.4524) (drill 0.2) (layers F.Cu B.Cu) (net 33))
   (segment (start 149.151206 89.071227) (end 149.151206 88.751332) (width 0.1545) (layer F.Cu) (net 33))
