File: breadbee.kicad_pcb (KiCad board)
At the start: 4 copper layers, 32 x 30 mm, 83 parts, among them J1 HR961160C, J2 Conn_02x12_Odd_Even, J3 USB_B_Micro, J4 Conn_01x21, U1 msc313e, U2 spinor, U3 ea3036c, U4 ch340e, U5 tvsarray, Y1 Crystal_GND24

Commit message: pcb/footprint: fix up the thin pins on the soc
Other:
- board text added: "breadbee rev1 ~dgp"
- board text removed: "breadbee rev0 ~dgp"
