File: slice_alltheios/slice_alltheios.sch (KiCad schematic (older format))
At the start: 2 parts, among them J1 Conn_01x21, J2 Conn_02x10_Odd_Even

Commit message: Fix solder mask.
Parts:
- J1: footprint Connector_PinHeader_1.00mm:PinHeader_1x21_P1.00mm_Vertical -> edgeconnector:breadbee_1mm_header_connector
Changed lines of the file:
@@
 EESchema Schematic File Version 4
+LIBS:slice_alltheios-cache
 EELAYER 29 0
 EELAYER END
@@
 F 0 "J1" H 4568 5067 50  0000 C CNN
 F 1 "Conn_01x21" H 4568 4976 50  0000 C CNN
-F 2 "Connector_PinHeader_1.00mm:PinHeader_1x21_P1.00mm_Vertical" H 4650 3850 50  0001 C CNN
+F 2 "edgeconnector:breadbee_1mm_header_connector" H 4650 3850 50  0001 C CNN
 F 3 "~" H 4650 3850 50  0001 C CNN
 	1    4650 3850
